Commit message: code used for benchmarking

File: assets/urdf/bittle/urdf/bittle.urdf (robot description, URDF)
Before this commit: robot bittle, 13 links, 12 joints
Links:
- link mainboard_link: mass 0.001 -> 0.025
Joints:
- joint left-back-knee-joint: limit lower=-1.22173 upper=1.48353 effort=15.0 velocity=1.5708 -> lower=-1.22173 upper=1.48353 effort=15 velocity=1.5708
- joint left-back-shoulder-joint: limit lower=-1.5708 upper=1.22173 effort=15.0 velocity=1.5708 -> lower=-1.5708 upper=1.22173 effort=15 velocity=1.5708
- joint left-front-knee-joint: limit lower=-1.22173 upper=1.48353 effort=15.0 velocity=1.5708 -> lower=-1.22173 upper=1.48353 effort=15 velocity=1.5708
- joint left-front-shoulder-joint: limit lower=-1.5708 upper=1.22173 effort=15.0 velocity=1.5708 -> lower=-1.5708 upper=1.22173 effort=15 velocity=1.5708
- joint right-back-knee-joint: limit lower=-1.22173 upper=1.48353 effort=15.0 velocity=1.5708 -> lower=-1.22173 upper=1.48353 effort=15 velocity=1.5708
- joint right-back-shoulder-joint: limit lower=-1.5708 upper=1.22173 effort=15.0 velocity=1.5708 -> lower=-1.5708 upper=1.22173 effort=15 velocity=1.5708
- joint right-front-knee-joint: limit lower=-1.22173 upper=1.48353 effort=15.0 velocity=1.5708 -> lower=-1.22173 upper=1.48353 effort=15 velocity=1.5708
- joint right-front-shoulder-joint: limit lower=-1.5708 upper=1.22173 effort=15.0 velocity=1.5708 -> lower=-1.5708 upper=1.22173 effort=15 velocity=1.5708
