Commit message: fixed effort in urdf

File: assets/urdf/atlas/urdf/atlas_v4_with_multisense.urdf (robot description, URDF)
Before this commit: robot multisense_sl, 31 links, 30 joints
Joints:
- joint r_leg_aky: limit lower=-1 upper=0.7 effort=92 velocity=12 -> lower=-1 upper=0.7 effort=92

Commit message: reworked obs collection used default motion files still using old T pose

File: assets/urdf/atlas/urdf/atlas_v4_with_multisense.urdf (robot description, URDF)
Before this commit: robot multisense_sl, 31 links, 30 joints
Links:
- link utorso: mass 84.409 -> 0.409
